Commit message: Working on xacro,xml,gazebo convert.... weird directions

File: urdf/robot.xacro (robot description, xacro)
@@ -1,71 +1,4 @@
 <?xml version="1.0" ?>
 <robot name="robot">
-    <gazebo reference="joint_chassis_caster_wheel">
-        <preserveFixedJoint>true</preserveFixedJoint>
-    </gazebo>
-    <gazebo reference="link_chassis">
-        <material>Gazebo/TurquoiseGlow</material>
-    </gazebo>
-    <gazebo reference="link_caster_wheel">
-        <material>Gazebo/Blue</material>
-        <mu1>0</mu1>
-        <mu2>0</mu2>
-    </gazebo>
-    <gazebo reference="link_left_wheel">
-        <material>Gazebo/Wood</material>
-        <mu1>1</mu1>
-        <mu2>1</mu2>
-    </gazebo>
-    <gazebo reference="link_right_wheel">
-        <material>Gazebo/Wood</material>
-        <mu1>1</mu1>
-        <mu2>1</mu2>
-    </gazebo>
-    <gazebo>
-        <plugin filename="libgazebo_ros_diff_drive.so" name="differential_drive_controller">
-            <alwaysOn>true</alwaysOn>
-            <updateRate>20</updateRate>
-            <leftJoint>joint_chassis_left_wheel</leftJoint>
-            <rightJoint>joint_chassis_right_wheel</rightJoint>
-            <wheelSeparation>1.66</wheelSeparation>
-            <wheelDiameter>0.8</wheelDiameter>
-            <torque>10</torque>
-            <commandTopic>cmd_vel</commandTopic>
-            <odometryTopic>odom</odometryTopic>
-            <odometryFrame>odom</odometryFrame>
-            <robotBaseFrame>link_chassis</robotBaseFrame>
-        </plugin>
-    </gazebo>
-    <gazebo reference="link_laser_scan">
-        <sensor type="ray" name="head_hokuyo_sensor">
-            <pose>0 0 0 0 0 0</pose>
-            <visualize>true</visualize>
-            <update_rate>20</update_rate>
-            <ray>
-                <scan>
-                    <horizontal>
-                        <samples>720</samples>
-                        <resolution>1</resolution>
-                        <min_angle>-1.570796</min_angle>
-                        <max_angle>1.570796</max_angle>
-                    </horizontal>
-                </scan>
-                <range>
-                    <min>0.20</min>
-                    <max>10.0</max>
-                    <resolution>0.01</resolution>
-                </range>
-                <noise>
-                    <type>gaussian</type>
-                    <mean>0.0</mean>
-                    <stddev>0.01</stddev>
-                </noise>
-            </ray>
-            <plugin name="gazebo_ros_head_hokuyo_controller" filename="libgazebo_ros_laser.so">
-                <topicName>/laser/scan</topicName>
-                <frameName>sensor_laser</frameName>
-            </plugin>
-        </sensor>
-    </gazebo>
     <!-- Link - chassis -->
     <link name="link_chassis">
@@ -254,11 +187,4 @@
         </visual>
     </link>
-    <!-- Gazebo tags - Laser scan -->
-<gazebo reference="joint_laser_scan_chassis">
-    <preserveFixedJoint>true</preserveFixedJoint>
-</gazebo>
-<gazebo reference="link_laser_scan">
-    <material>Gazebo/DarkGrey</material>
-</gazebo>
     <!-- Laser scan -->
     <joint name="joint_laser_scan_chassis" type="fixed">

Commit message: sorted through the alterations for the xacro conversion

File: urdf/robot.xacro (robot description, xacro)
@@ -1,4 +1,8 @@
 <?xml version="1.0" ?>
-<robot name="robot">
+<robot name="robot" xmlns:xacro="http://www.ros.org/wiki/xacro">
+    <xacro:include filename="$(find robot_description)/urdf/robot.gazebo" />
+    <!-- Parameters -->
+    <xacro:property name="chassis_mass" value="10" />
+    <xacro:property name="pi" value="3.1415926535897931"/>
     <!-- Link - chassis -->
     <link name="link_chassis">

Commit message: XML parsing error: mismatched tag: line 85, column 2: inside xacro file

File: urdf/robot.xacro (robot description, xacro)
@@ -220,3 +220,43 @@
         </collision>
     </link>
+    <!-- Robot tail -->
+    <joint name="joint_tail" type="continuous">
+        <origin rpy="0 0 0" xyz="-1 0 0" />
+        <child link="link_tail" />
+        <axis rpy="0 0 0" xyz="0 1 0" />
+        <parent link="link_chassis" />
+        <joint_properties damping="1.0" friction="1.0" />
+    </joint>
+    <link name="link_tail">
+        <inertial>
+            <origin xyz="0 0 0" rpy="0 0 0" />
+            <mass value="0.5" />
+            <inertia ixx="0.000252666666667" ixy="0" ixz="0" iyy="0.000252666666667" iyz="0" izz="0.0005"/>
+        </inertial>
+        <visual>
+            <origin xyz="-0.2 0 0" rpy="0 ${pi/2} 0" />
+            <geometry>
+                <cylinder radius="0.05" length="0.40"/>
+            </geometry>
+            <material name="Red">
+                <color rgba="0.7 0.1 0.1 1" />
+            </material>
+        </visual>
+        <collision>
+            <origin xyz="-0.2 0 0" rpy="0 ${pi/2} 0"/>
+            <geometry>
+                <cylinder radius="0.05" length="0.40"/>
+            </geometry>
+        </collision>
+    </link>
+<transmission name="tran_tail">
+    <type>transmission_interface/SimpleTransmission</type>
+    <joint name="joint_tail">
+        <hardwareInterface>hardware_interface/EffortJointInterface</hardwareInterface>
+    </joint>
+    <actuator name="motor_joint_tail">
+        <hardwareInterface>hardware_interface/EffortJointInterface</hardwareInterface>
+        <mechanicalReduction>1</mechanicalReduction>
+    </actuator>
+</transmission>
 </robot>
